Commit message: Fix: Límite superior J5

File: urdf/r6g_steppermotor.urdf (robot description, URDF)
Before this commit: robot r6g_steppermotor, 7 links, 6 joints
Joints:
- joint Joint5: limit lower=-0.1745329 upper=1.57079632 effort=0 velocity=0 -> lower=-0.1745329 upper=1.74532925 effort=0 velocity=0
